File: KiCAD/epaper-adapters/feather_epaper_adapter.kicad_pcb (KiCad board)
At the start: 2 copper layers, 50.8 x 22.9 mm, 20 parts, among them J2 Adafruit_Feather_Conn, J3 SPI_conn, P1 MOLEX_FPC_RCPT_24POS, Q1 IRLML6344TRPBF / SI1308EDL

Commit message: epaper-adapters: feather_epaper_adapter rev 1.0
Parts:
- Q1: footprint TO_SOT_Packages_SMD:SOT-323_SC-70 -> TO_SOT_Packages_SMD:SOT-23
- moved Q1 0.24 mm to (148.1, 108.7)
Routing:
- net /RESE: track 19.6 -> 24.1 mm
- net /SW: track 17.7 -> 18.8 mm
- net /GDR: track 23.9 -> 24.4 mm
Other:
- board text added: ">|"
- board text added: "Adafruit Feather ePaper Wing Rev 1.0 Sat Mar 24, 2018 @hanyazou"
- board text added: "ePaper Wing for Adafruit Feather Rev 1.0 Sat Mar 24, 2018 @hanyazou"
- board text added: "|<"
- board text removed: "Adafruit Feather ePaper Adapter Rev 0.9 Sun Mar 18, 2018 @hanyazou"
- board text removed: "ePaper Adapter for Adafruit Feather Rev 0.9 Sun Mar 18, 2018 @hanyazou"
