File: KiCAD/Hanyaduino-nRF52/Adafruit nRF52 Bluefruit Feather.kicad_pcb (KiCad board)
At the start: 2 copper layers, 34.7 x 17.8 mm, 37 parts, among them J1 Conn_01x02_Male, J2 Arduino_pro_micro_conn, J3 USB_B_Micro, J4 Conn_01x04_Male, Q1 DMG3415U, U1 MCP73831-2-OT, U2 NRF52832_MODULE_MDBT42, U3 CP2104, U4 AP2113(3.3V), Y1 32.768KHz

Commit message: Hanyaduino nRF52 v0.81
Parts:
- moved J4 6.67 mm to (141.6, 127.9)
Routing:
- net GND: track 126.6 -> 127.7 mm, vias 17 -> 18
- net SWCLK: track 11.9 -> 12.1 mm, vias 1 -> 2
- net SWDIO: track 12.3 -> 12.6 mm, vias 1 -> 2
- net VCC: track 77.9 -> 78.0 mm, vias 11 -> 12
Other:
- board text added: "Hanyaduino nRF52 v0.81 Nov 10, 2018"
- board text removed: "Hanyaduino nRF52 v0.8 Nov 10, 2018"
Changed lines of the file:
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@@
   (general
     (thickness 1.6)
-    (drawings 32)
-    (tracks 1140)
+    (drawings 34)
+    (tracks 1149)
     (zones 0)
     (modules 37)
@@
   )
   (module "library:Conn4 1.0mm pitch" (layer F.Cu)
-    (at 141.605 121.2215)
+    (at 141.589 127.889)
     (fp_text reference J4 (at -0.635 6.7945) (layer F.SilkS)
       (effects (font (size 1 1) (thickness 0.15)))
@@
     )
   )
+  (gr_poly (pts (xy 140.335 121.158) (xy 143.8275 121.158) (xy 143.8275 121.666) (xy 140.335 121.666)) (layer F.Mask) (width 0.15))
+  (gr_poly (pts (xy 140.335 121.158) (xy 143.8275 121.158) (xy 143.8275 121.666) (xy 140.335 121.666)) (layer B.Mask) (width 0.15))
   (dimension 17.907113 (width 0.3) (layer B.SilkS)
     (gr_text "17.907 mm" (at 156.436672 115.480814 -89.79682433) (layer B.SilkS)
@@
     (effects (font (size 0.6 0.6) (thickness 0.15)))
   )
-  (gr_text "Hanyaduino nRF52 v0.8\nNov 10, 2018" (at 146.3675 114.9985 90) (layer B.SilkS)
+  (gr_text "Hanyaduino nRF52 v0.81\nNov 10, 2018" (at 146.3675 114.9985 90) (layer B.SilkS)
     (effects (font (size 0.9 0.8) (thickness 0.125)) (justify mirror))
   )
@@
   (segment (start 144.37 111.57) (end 144.37 111.243) (width 0.381) (layer F.Cu) (net 2))
   (segment (start 144.37 119.57) (end 144.37 120.012) (width 0.381) (layer F.Cu) (net 2))
-  (segment (start 144.748 122.174) (end 143.732 121.158) (width 0.381) (layer F.Cu) (net 2))
   (segment (start 145.504 122.174) (end 144.748 122.174) (width 0.381) (layer F.Cu) (net 2))
-  (segment (start 144.513 120.277) (end 143.732 121.058) (width 0.381) (layer F.Cu) (net 2))
   (segment (start 144.37 119.57) (end 144.513 119.713) (width 0.381) (layer F.Cu) (net 2))
   (segment (start 144.513 119.713) (end 144.513 120.277) (width 0.381) (layer F.Cu) (net 2))
-  (segment (start 143.732 121.058) (end 143.732 121.158) (width 0.381) (layer F.Cu) (net 2))
   (segment (start 133.552 111.72) (end 133.338 111.506) (width 0.381) (layer F.Cu) (net 2))
   (segment (start 134.62 111.72) (end 133.552 111.72) (width 0.381) (layer F.Cu) (net 2))
@@
   (segment (start 134.633992 111.125008) (end 134.643067 111.125008) (width 0.381) (layer F.Cu) (net 2))
   (segment (start 135.470899 111.467907) (end 135.128 111.125008) (width 0.381) (layer B.Cu) (net 2))
+  (via (at 143.51 121.412) (size 0.6858) (drill 0.3302) (layers F.Cu B.Cu) (net 2))
+  (segment (start 144.37 120.552) (end 143.51 121.412) (width 0.381) (layer F.Cu) (net 2))
+  (segment (start 144.37 119.57) (end 144.37 120.552) (width 0.381) (layer F.Cu) (net 2))
+  (segment (start 144.328899 121.754899) (end 143.852899 121.754899) (width 0.381) (layer F.Cu) (net 2))
+  (segment (start 143.852899 121.754899) (end 143.51 121.412) (width 0.381) (layer F.Cu) (net 2))
+  (segment (start 144.748 122.174) (end 144.328899 121.754899) (width 0.381) (layer F.Cu) (net 2))
   (segment (start 120.96172 121.14022) (end 120.9795 121.158) (width 0.381) (layer F.Cu) (net 3))
   (segment (start 120.01246 121.14022) (end 120.96172 121.14022) (width 0.381) (layer F.Cu) (net 3))
@@
   (segment (start 137.421798 121.40196) (end 137.764697 121.059061) (width 0.381) (layer F.Cu) (net 4))
   (segment (start 137.16 121.412) (end 137.411758 121.412) (width 0.381) (layer F.Cu) (net 4))
-  (segment (start 139.983149 121.481323) (end 140.339765 121.124707) (width 0.381) (layer B.Cu) (net 4))
   (segment (start 138.186959 121.481323) (end 137.764697 121.059061) (width 0.381) (layer B.Cu) (net 4))
   (segment (start 139.983149 121.481323) (end 138.186959 121.481323) (width 0.381) (layer B.Cu) (net 4))
@@
   (segment (start 134.4135 110.0455) (end 133.5325 110.0455) (width 0.381) (layer F.Cu) (net 4))
   (segment (start 133.408812 110.169188) (end 133.408812 110.635676) (width 0.381) (layer F.Cu) (net 4))
+  (via (at 140.589 121.412) (size 0.6858) (drill 0.3302) (layers F.Cu B.Cu) (net 4))
+  (segment (start 140.052472 121.412) (end 140.589 121.412) (width 0.381) (layer B.Cu) (net 4))
+  (segment (start 139.983149 121.481323) (end 140.052472 121.412) (width 0.381) (layer B.Cu) (net 4))
   (segment (start 131.838 111.584) (end 131.838 111.506) (width 0.1524) (layer F.Cu) (net 5))
   (segment (start 133.034 112.78) (end 131.838 111.584) (width 0.1524) (layer F.Cu) (net 5))
@@
   (segment (start 141.5415 120.948061) (end 143.398462 119.091099) (width 0.1524) (layer B.Cu) (net 42))
   (segment (start 143.001586 116.487293) (end 143.001586 114.084503) (width 0.1524) (layer B.Cu) (net 42))
-  (segment (start 141.5415 121.158) (end 141.5415 120.948061) (width 0.1524) (layer B.Cu) (net 42))
   (segment (start 143.398462 119.091099) (end 143.398462 116.884169) (width 0.1524) (layer B.Cu) (net 42))
   (segment (start 143.001586 114.084503) (end 143.344485 113.741604) (width 0.1524) (layer B.Cu) (net 42))
   (segment (start 143.398462 116.884169) (end 143.001586 116.487293) (width 0.1524) (layer B.Cu) (net 42))
+  (via (at 141.5415 121.412) (size 0.6858) (drill 0.3302) (layers F.Cu B.Cu) (net 42))
+  (segment (start 141.5415 120.948061) (end 141.5415 121.412) (width 0.1524) (layer B.Cu) (net 42))
   (via (at 143.33219 112.765312) (size 0.6858) (drill 0.3302) (layers F.Cu B.Cu) (net 43))
   (segment (start 143.309375 112.742497) (end 143.33219 112.765312) (width 0.1524) (layer F.Cu) (net 43))
@@
   (segment (start 143.703273 116.757913) (end 143.703273 119.217355) (width 0.1524) (layer B.Cu) (net 43))
   (segment (start 143.703273 119.217355) (end 142.5415 120.379128) (width 0.1524) (layer B.Cu) (net 43))
-  (segment (start 142.5415 120.379128) (end 142.5415 121.158) (width 0.1524) (layer B.Cu) (net 43))
   (segment (start 143.332188 116.386828) (end 143.703273 116.757913) (width 0.1524) (layer B.Cu) (net 43))
+  (via (at 142.5575 121.412) (size 0.6858) (drill 0.3302) (layers F.Cu B.Cu) (net 43))
+  (segment (start 142.5575 120.395128) (end 142.5575 121.412) (width 0.1524) (layer B.Cu) (net 43))
+  (segment (start 142.5415 120.379128) (end 142.5575 120.395128) (width 0.1524) (layer B.Cu) (net 43))
   (segment (start 135.87 119.57) (end 135.87 118.671667) (width 0.1524) (layer F.Cu) (net 44))
   (via (at 135.993451 118.548216) (size 0.6858) (drill 0.3302) (layers F.Cu B.Cu) (net 44))
@@
   (segment (start 120.719433 109.078601) (end 121.229143 109.588311) (width 0.1524) (layer B.Cu) (net 48))
   (segment (start 125.474003 109.588311) (end 125.535803 109.650111) (width 0.1524) (layer B.Cu) (net 48))
-  (via (at 144.954954 120.909436) (size 0.6858) (drill 0.3302) (layers F.Cu B.Cu) (net 49))
-  (segment (start 144.96039 120.904) (end 144.954954 120.909436) (width 0.1524) (layer F.Cu) (net 49))
   (segment (start 139.37 110.511946) (end 139.243366 110.385312) (width 0.1524) (layer F.Cu) (net 49))
   (segment (start 139.37 111.57) (end 139.37 110.511946) (width 0.1524) (layer F.Cu) (net 49))
   (via (at 139.243366 110.385312) (size 0.6858) (drill 0.3302) (layers F.Cu B.Cu) (net 49))
-  (segment (start 145.802564 120.909436) (end 145.808 120.904) (width 0.1524) (layer F.Cu) (net 49))
-  (segment (start 144.954954 120.909436) (end 145.802564 120.909436) (width 0.1524) (layer F.Cu) (net 49))
   (segment (start 139.026877 116.001793) (end 138.760178 116.268492) (width 0.1524) (layer B.Cu) (net 49))
   (segment (start 139.424362 114.251249) (end 139.192024 114.483586) (width 0.1524) (layer B.Cu) (net 49))
@@
   (segment (start 138.760178 116.268492) (end 138.830528 116.268492) (width 0.1524) (layer F.Cu) (net 49))
   (segment (start 138.830528 116.268492) (end 140.318846 117.75681) (width 0.1524) (layer F.Cu) (net 49))
-  (segment (start 144.954954 117.16377) (end 144.246589 116.455405) (width 0.1524) (layer B.Cu) (net 49))
-  (segment (start 144.954954 120.909436) (end 144.954954 117.16377) (width 0.1524) (layer B.Cu) (net 49))
   (segment (start 140.681299 117.75681) (end 141.140922 117.297187) (width 0.1524) (layer F.Cu) (net 49))
   (segment (start 140.318846 117.75681) (end 140.681299 117.75681) (width 0.1524) (layer F.Cu) (net 49))
-  (segment (start 144.246589 116.455405) (end 143.90369 116.112506) (width 0.1524) (layer B.Cu) (net 49))
   (segment (start 141.140922 117.297187) (end 141.751693 117.297187) (width 0.1524) (layer F.Cu) (net 49))
   (segment (start 142.936374 116.112506) (end 143.418757 116.112506) (width 0.1524) (layer F.Cu) (net 49))
   (via (at 143.90369 116.112506) (size 0.6858) (drill 0.3302) (layers F.Cu B.Cu) (net 49))
+  (segment (start 143.90369 116.112506) (end 144.955206 117.164022) (width 0.1524) (layer B.Cu) (net 49))
+  (via (at 144.955206 120.90959) (size 0.6858) (drill 0.3302) (layers F.Cu B.Cu) (net 49))
+  (segment (start 144.960796 120.904) (end 144.955206 120.90959) (width 0.1524) (layer F.Cu) (net 49))
+  (segment (start 144.955206 120.909184) (end 144.955206 120.90959) (width 0.1524) (layer F.Cu) (net 49))
+  (segment (start 144.955206 117.164022) (end 144.955206 120.424657) (width 0.1524) (layer B.Cu) (net 49))
+  (segment (start 144.96039 120.904) (end 144.955206 120.909184) (width 0.1524) (layer F.Cu) (net 49))
+  (segment (start 145.808 120.904) (end 144.960796 120.904) (width 0.1524) (layer F.Cu) (net 49))
+  (segment (start 144.955206 120.424657) (end 144.955206 120.90959) (width 0.1524) (layer B.Cu) (net 49))
   (segment (start 115.505056 120.2175) (end 115.543528 120.179028) (width 0.1524) (layer F.Cu) (net 50))
   (via (at 115.543528 120.179028) (size 0.6858) (drill 0.3302) (layers F.Cu B.Cu) (net 50))
