File: KiCAD/SAMD21/SAMD21.sch (KiCad schematic (older format))
At the start: 32 parts, among them IC1 ATSAMD21E18A-AU, IC2 ATSAMD21G18, J1 USB_OTG, J2 CortexDebugConn10, J3 Arduino_pro_micro_conn, J4 Conn_02x04_Odd_Even, J5 CONN_01X04, J6 Groveconn4, U1 WS2812B, U2 TLV71333PDBV, U3 W25Q32, Y1 32.768kHz

Commit message: updated
Parts:
- removed J1: USB_OTG, library:USB_Micro-B_Molex_47346-0001, symbol USB_OTG
- removed J4: Conn_02x04_Odd_Even, Pin_Headers:Pin_Header_Straight_2x04_Pitch2.54mm, symbol Conn_02x04_Odd_Even
- removed J5: CONN_01X04, Pin_Headers:Pin_Header_Straight_1x04_Pitch1.27mm, symbol Conn_01x04
- removed U2: TLV71333PDBV, TO_SOT_Packages_SMD:SOT-23-5_HandSoldering, symbol TLV71333PDBV
- added J1: USB_B_Micro, symbol Connector:USB_B_Micro
- added J4: Conn_02x04_Odd_Even, symbol Connector_Generic:Conn_02x04_Odd_Even
- added J5: Conn_01x04_Male, symbol Connector:Conn_01x04_Male
- added U2: TLV71333PDBV, Package_TO_SOT_SMD:SOT-23-5, symbol Regulator_Linear:TLV71333PDBV
- C1, C2, C3, C4, C5, C6, C7: symbol C_Small -> Device:C_Small
- D1, D2, D3, D4: symbol LED -> Device:LED
- IC1: symbol ATSAMD21E18A-AU -> mylib:ATSAMD21E18A-AU
- IC2: symbol ATSAMD21G18 -> mylib:ATSAMD21G18
- J2: symbol CortexDebugConn10 -> mylib:CortexDebugConn10
- J3: symbol Arduino_pro_micro_conn -> mylib:Arduino_pro_micro_conn
- J6: symbol Groveconn4 -> mylib:Groveconn4
- JP1: symbol Jumper_NO_Small -> Device:Jumper_NO_Small
- R1, R2, R3, R4, R5, R6, R7: symbol R -> Device:R
- S1: symbol tactile_switch -> mylib:tactile_switch
- U1: symbol WS2812B -> mylib:WS2812B
- U3: symbol W25Q32 -> mylib:W25Q32
- Y1: symbol Crystal_Small -> Device:Crystal_Small
Connections:
- wire segments 215 -> 238
