File: KiCAD/Hanyaduino-nRF52840/Hanyaduino-nRF52840.sch (KiCad schematic (older format))
At the start: 43 parts, among them J1 Conn_01x02_Male, J2 Arduino_pro_micro_conn, J3 USB_B_Micro, J4 Conn_01x04_Male, Q1 DMG3415U, U1 MCP73831-2-OT, U2 NRF52832_MODULE_MDBT42, U3 nRF52840, U4 AP2113(3.3V), Y1 32.768KHz

Commit message: Add neopixel and delete crystal
Parts:
- removed C1: 1uF, Capacitors_SMD:C_0603, symbol Adafruit_nRF52_Bluefruit_Feather-eagle-import:CAP_CERAMIC0603_NO
- removed C11, C8: 10uF, Capacitors_SMD:C_0603, symbol Device:C_Small
- removed C14: 1nF, Capacitors_SMD:C_0603, symbol Adafruit_nRF52_Bluefruit_Feather-eagle-import:CAP_CERAMIC0603_NO
- removed C4, C5: 22pF, Capacitors_SMD:C_0603, symbol Adafruit_nRF52_Bluefruit_Feather-eagle-import:CAP_CERAMIC0603_NO
- removed C6, C7: 300pF, Capacitors_SMD:C_0603, symbol Adafruit_nRF52_Bluefruit_Feather-eagle-import:CAP_CERAMIC_0603MP
- removed D2: CHG, LEDs:LED_0603, symbol Device:LED
- removed D7: PWR LED, LEDs:LED_0603, symbol Device:LED
- removed J1: Conn_01x02_Male, Connectors_JST:JST_PH_B2B-PH-SM4-TB_02x2.00mm_Straight, symbol Connector:Conn_01x02_Male
- removed J4: Conn_01x04_Male, library:Conn4 1.0mm pitch, symbol Connector:Conn_01x04_Male
- removed JP1, JP2: Conn_01x01_Female, Connectors:1pin, symbol Connector:Conn_01x01_Female
- removed L1: 10uH, Inductors_SMD:L_0805, symbol Adafruit_nRF52_Bluefruit_Feather-eagle-import:INDUCTOR0805-NO
- removed MS1: FEATHERWING, library:Adafruit_Feather_board, symbol Adafruit_nRF52_Bluefruit_Feather-eagle-import:FEATHERWING
- removed R12: 100K, Resistors_SMD:R_0603, symbol Device:R
- removed R13: 10K, Resistors_SMD:R_0603, symbol Device:R
- removed R4: 1K, Resistors_SMD:R_0603, symbol Adafruit_nRF52_Bluefruit_Feather-eagle-import:RESISTOR_0603_NOOUT
- removed R8: 2M, Resistors_SMD:R_0603, symbol Adafruit_nRF52_Bluefruit_Feather-eagle-import:RESISTOR_0603_NOOUT
- removed S2: DFU SW, library:B3U-1000P(OMRON Ultra-small Tactile Switch), symbol mylib:tactile_switch
- removed U2: NRF52832_MODULE_MDBT42, library:MDBT42, symbol mylib:NRF52832_MODULE_MDBT42
- removed U3: nRF52840, BL654-nRF52840-451-00001:XCVR_451-00001, symbol MCU_Nordic:nRF52840
- added C1, C5: 10uF, Capacitors_SMD:C_0603, symbol Device:C_Small
- added C2: 22pF, Capacitors_SMD:C_0603, symbol Adafruit_nRF52_Bluefruit_Feather-eagle-import:CAP_CERAMIC0603_NO
- added C6: 1nF, Capacitors_SMD:C_0603, symbol Adafruit_nRF52_Bluefruit_Feather-eagle-import:CAP_CERAMIC0603_NO
- added D1: CHG, LEDs:LED_0603, symbol Device:LED
- added D6: PWR LED, LEDs:LED_0603, symbol Device:LED
- added D7: SK6812, KiCAD footprints:LED_SK6812MINI_PLCC4_3.5x3.5mm_P1.75mm, symbol LED:WS2812B
- added J1: Conn_01x02_Female, library:3 point pad, symbol Connector:Conn_01x02_Female
- added J3: Conn_01x02_Male, Connectors_JST:JST_PH_B2B-PH-SM4-TB_02x2.00mm_Straight, symbol Connector:Conn_01x02_Male
- added J5: Conn_01x04_Male, library:Conn4 1.0mm pitch, symbol Connector:Conn_01x04_Male
- added R4: 100K, Resistors_SMD:R_0603, symbol Device:R
- added R5: 10K, Resistors_SMD:R_0603, symbol Device:R
- added R7: 2M, Resistors_SMD:R_0603, symbol Adafruit_nRF52_Bluefruit_Feather-eagle-import:RESISTOR_0603_NOOUT
- added R8: 10k, Resistors_SMD:R_0603, symbol Device:R
- added R9: 1K, Resistors_SMD:R_0603, symbol Adafruit_nRF52_Bluefruit_Feather-eagle-import:RESISTOR_0603_NOOUT
- added U2: NRF52840_MODULE_BL654_451-00001, BL654-nRF52840-451-00001:XCVR_451-00001, symbol mylib:NRF52840_MODULE_BL654_451-00001
- added U4: W25Q32, Housings_SOIC:SOIJ-8_5.3x5.3mm_Pitch1.27mm, symbol mylib:W25Q32
- C3: value 10uF -> 22pF
- renumbered C2 to C4, D3 to D2, D1 to D3, D9 to D5, J3 to J4, R14 to R10, U4 to U3
Connections:
- net labels added: D0/TX, D1/RX, D10, D11/TX, D12/RX, D13, D14/A0, D15/A1, D16/A2, D17/A3, D18/A4, D19/A5, D2, D20/A6(Battery), D21/A7(ARef), D22/SDA(I2C), D23/SCL(I2C), D24/MISO(SPI), D25/MOSI(SPI), D26/SCK(SPI), D27/CLK(QSPI), D28/CS(QSPI), D29/data0(QSPI), D3/LED1, D30/data1(QSPI), D31/data2(QSPI), D32/data3(QSPI), D33, D35, D36, D37, D38, D39, D4/LED2, D43, D44, D45, D46, D6, D7(button), D8/NeoPixel, XL1, XL2
- net labels removed: 3.3V, A0, A0/0.02, A1, A1/0.03, A2, A2/0.04, A3, A3/0.05, A4, A4/0.28, A5, A5/0.29, A6/P0.30, A7/P0.31, D10/SS, D11, D12, D4/A6, D6/A7, D7, D8/A8, DFU, EN, FRST, LED1, LED2, MISO, MOSI, P0.07, P0.09/NFC1, P0.10/NFC2, P0.11, P0.15, P0.16, P0.27, RX, RXD, SCK, SCL, SDA, SWO, TX, TXD
- wire segments 224 -> 223
- no-connect marks 8 -> 23
Other:
- note added: "Arduino pro micro compatible pins"
- note added: "BL654 nRF52840 module"
- note added: "Battery connector"
- note added: "Debug connector"
- note added: "Optional 32.768kHz Crystal"
- note added: "RESET\nSWITCH"
- note added: "SPI flash"
- note added: "UART connector"
- note added: "USB connector"
- note removed: "Adafruit Feather\nPinout"
- note removed: "Debug connector (small)"

Commit message: layout
Parts:
- removed J1: Conn_01x02_Female, library:3 point pad, symbol Connector:Conn_01x02_Female
- added J1: Conn_01x03_Female, library:3 point pad, symbol Connector:Conn_01x03_Female
Connections:
- wire segments 223 -> 225
Changed lines of the file:
@@
 Wire Wire Line
 	1750 8150 1500 8150
-$Comp
-L Connector:Conn_01x02_Female J1
-U 1 1 5EB8FCEE
-P 1950 8050
-F 0 "J1" H 1977 8026 50  0000 L CNN
-F 1 "Conn_01x02_Female" H 1977 7935 50  0000 L CNN
-F 2 "library:3 point pad" H 1950 8050 50  0001 C CNN
-F 3 "~" H 1950 8050 50  0001 C CNN
-	1    1950 8050
-	1    0    0    -1
-$EndComp
 Text Notes 1300 3050 0    59   ~ 0
 BL654 nRF52840 module
@@
 Wire Wire Line
 	6100 8550 6100 8450
+$Comp
+L Connector:Conn_01x03_Female J1
+U 1 1 5C0E47FD
+P 1950 8150
+F 0 "J1" H 1977 8176 50  0000 L CNN
+F 1 "Conn_01x03_Female" H 1977 8085 50  0000 L CNN
+F 2 "library:3 point pad" H 1950 8150 50  0001 C CNN
+F 3 "~" H 1950 8150 50  0001 C CNN
+	1    1950 8150
+	1    0    0    -1
+$EndComp
+$Comp
+L power:GND #PWR016
+U 1 1 5C0E4D20
+P 1450 8350
+F 0 "#PWR016" H 1450 8100 50  0001 C CNN
+F 1 "GND" H 1450 8200 50  0000 C CNN
+F 2 "" H 1450 8350 50  0001 C CNN
+F 3 "" H 1450 8350 50  0001 C CNN
+	1    1450 8350
+	1    0    0    -1
+$EndComp
+Wire Wire Line
+	1450 8350 1450 8250
+Wire Wire Line
+	1450 8250 1750 8250
 $EndSCHEMATC

Commit message: Hanyaduino-nRF52840 v1.0
Parts:
- removed D7: SK6812, KiCAD footprints:LED_SK6812MINI_PLCC4_3.5x3.5mm_P1.75mm, symbol LED:WS2812B
- added D7: SK6812MINI, LED_SMD:LED_SK6812MINI_PLCC4_3.5x3.5mm_P1.75mm, symbol LED:SK6812MINI
Connections:
- wire segments 225 -> 223
- no-connect marks 23 -> 21
Changed lines of the file:
@@
 Text GLabel 4400 6050 2    50   Input ~ 0
 D17/A3
-Text GLabel 5950 5600 2    50   Input ~ 0
+Text GLabel 6300 4150 0    50   Input ~ 0
 D18/A4
-Text GLabel 5950 5700 2    50   Input ~ 0
+Text GLabel 6300 4550 0    50   Input ~ 0
 D19/A5
 Text GLabel 4400 5950 2    50   Input ~ 0
@@
 Text GLabel 6300 3550 0    50   Input ~ 0
 D0/TX
-Text GLabel 6300 4150 0    50   Input ~ 0
-D4/LED2
 Text GLabel 6300 4250 0    50   Input ~ 0
 D5
@@
 Text GLabel 6300 4450 0    50   Input ~ 0
 D7(button)
-Text GLabel 6300 4550 0    50   Input ~ 0
-D8/NeoPixel
 Text GLabel 6300 4650 0    50   Input ~ 0
 D9
@@
 Text GLabel 1600 4850 0    50   Input ~ 0
 D19/A5
-NoConn ~ 5800 5600
-NoConn ~ 5800 5700
 NoConn ~ 5800 5900
 NoConn ~ 5800 6100
@@
 Wire Wire Line
 	5950 5900 5800 5900
-Wire Wire Line
-	5950 5700 5800 5700
-Wire Wire Line
-	5800 5600 5950 5600
 Text GLabel 6300 3850 0    39   Input ~ 0
 GND
@@
 Text Notes 5800 3200 0    59   ~ 0
 Arduino pro micro compatible pins
-$Comp
-L LED:WS2812B D7
-U 1 1 5C0CEFA0
-P 6100 8150
-F 0 "D7" H 6441 8196 50  0000 L CNN
-F 1 "SK6812" H 6441 8105 50  0000 L CNN
-F 2 "KiCAD footprints:LED_SK6812MINI_PLCC4_3.5x3.5mm_P1.75mm" H 6150 7850 50  0001 L TNN
-F 3 "https://cdn-shop.adafruit.com/datasheets/WS2812B.pdf" H 6200 7775 50  0001 L TNN
-	1    6100 8150
-	1    0    0    -1
-$EndComp
 Text GLabel 5550 8150 0    50   Input ~ 0
 D8/NeoPixel
@@
 Wire Wire Line
 	1450 8250 1750 8250
+$Comp
+L LED:SK6812MINI D7
+U 1 1 5C16FBFC
+P 6100 8150
+F 0 "D7" H 6441 8196 50  0000 L CNN
+F 1 "SK6812MINI" H 6441 8105 50  0000 L CNN
+F 2 "LED_SMD:LED_SK6812MINI_PLCC4_3.5x3.5mm_P1.75mm" H 6150 7850 50  0001 L TNN
+F 3 "https://cdn-shop.adafruit.com/product-files/2686/SK6812MINI_REV.01-1-2.pdf" H 6200 7775 50  0001 L TNN
+	1    6100 8150
+	1    0    0    -1
+$EndComp
 $EndSCHEMATC

Commit message: Hanyaduino nRF52840 v1.5
Connections:
- wire segments 223 -> 219
- no-connect marks 21 -> 19
Changed lines of the file:
@@
 Text GLabel 10650 4000 2    39   Input ~ 0
-VCC
-Text GLabel 9500 4200 0    39   Input ~ 0
 VCC
 Wire Wire Line
@@
 	9500 4300 9700 4300
 Wire Wire Line
-	10500 4000 10550 4000
-Wire Wire Line
-	10500 4100 10550 4100
-Wire Wire Line
-	10550 4100 10550 4000
-Connection ~ 10550 4000
-Wire Wire Line
 	10500 4200 10650 4200
 Wire Wire Line
@@
 Wire Wire Line
 	9600 4000 9700 4000
-Wire Wire Line
-	10550 4000 10650 4000
-Text GLabel 9500 4100 0    50   Input ~ 0
+Text GLabel 10650 4300 2    50   Input ~ 0
 D29/data0(QSPI)
 Text GLabel 10650 4200 2    50   Input ~ 0
@@
 Text GLabel 9500 4000 0    50   Input ~ 0
 D28/CS(QSPI)
-Text GLabel 10650 4300 2    50   Input ~ 0
+Text GLabel 9500 4100 0    50   Input ~ 0
 D30/data1(QSPI)
-Text GLabel 10650 4800 2    50   Input ~ 0
+Text GLabel 10650 4100 2    50   Input ~ 0
 D32/data3(QSPI)
-Text GLabel 10650 4700 2    50   Input ~ 0
+Text GLabel 9500 4200 0    50   Input ~ 0
 D31/data2(QSPI)
-NoConn ~ 10500 4800
-NoConn ~ 10500 4700
-Wire Wire Line
-	10500 4700 10650 4700
-Wire Wire Line
-	10650 4800 10500 4800
 Text Notes 850  7550 0    59   ~ 0
 UART connector
@@
 	1    0    0    -1
 $EndComp
+Wire Wire Line
+	10500 4000 10650 4000
+Wire Wire Line
+	10500 4100 10650 4100
 $EndSCHEMATC
