File: KiCAD/USB-swith/USB-switch.sch (KiCad schematic (older format))
At the start: 17 parts, among them Q1 AO3401A, U1 PIC12LF1840-ISN, U2 FSUSB42MUX, U3 AMS1117-3.3, U4 PI3USB302-AZBEX

Commit message: Add R5
Parts:
- added R5: 10k, symbol Device:R
Connections:
- net SW_IN: now also R5.2
- net VBUS: now also R5.1
Other:
- moved on the sheet: D1, D2, R4, S1
Changed lines of the file:
@@
 Wire Wire Line
 	4950 3750 5350 3750
-Text GLabel 7750 3350 0    50   Input ~ 0
-SEL
-$Comp
-L Device:R R2
-U 1 1 6153E959
-P 8300 4100
-F 0 "R2" H 8370 4146 50  0000 L CNN
-F 1 "55Ω" H 8370 4055 50  0000 L CNN
-F 2 "" V 8230 4100 50  0001 C CNN
-F 3 "~" H 8300 4100 50  0001 C CNN
-	1    8300 4100
-	1    0    0    -1
-$EndComp
-Text GLabel 8200 4350 0    50   Input ~ 0
-3V3
-Wire Wire Line
-	8200 4350 8300 4350
-Wire Wire Line
-	8300 4350 8300 4250
-Wire Wire Line
-	8300 3950 8300 3850
 $Comp
 L MCU_Microchip_PIC12:PIC12LF1840-ISN U1
@@
 L mylib:tactile_switch S1
 U 1 1 61562533
-P 5950 5400
-F 0 "S1" H 5950 5737 60  0000 C CNN
-F 1 "tactile_switch" H 5950 5631 60  0000 C CNN
-F 2 "" H 6150 5350 60  0001 C CNN
-F 3 "" H 6150 5350 60  0001 C CNN
-	1    5950 5400
+P 7950 5400
+F 0 "S1" H 7950 5737 60  0000 C CNN
+F 1 "tactile_switch" H 7950 5631 60  0000 C CNN
+F 2 "" H 8150 5350 60  0001 C CNN
+F 3 "" H 8150 5350 60  0001 C CNN
+	1    7950 5400
 	1    0    0    -1
 $EndComp
@@
 Wire Wire Line
 	8650 2000 8750 2000
-Text GLabel 7750 3650 0    50   Input ~ 0
-GP4
-Wire Wire Line
-	7750 3650 8000 3650
 $Comp
 L Device:LED D1
 U 1 1 61593E76
-P 8400 4850
-F 0 "D1" H 8393 4595 50  0000 C CNN
-F 1 "LED" H 8393 4686 50  0000 C CNN
-F 2 "" H 8400 4850 50  0001 C CNN
-F 3 "~" H 8400 4850 50  0001 C CNN
-	1    8400 4850
+P 2300 4950
+F 0 "D1" H 2293 4695 50  0000 C CNN
+F 1 "LED" H 2293 4786 50  0000 C CNN
+F 2 "" H 2300 4950 50  0001 C CNN
+F 3 "~" H 2300 4950 50  0001 C CNN
+	1    2300 4950
 	-1   0    0    1
 $EndComp
-Text GLabel 7750 4850 0    50   Input ~ 0
+Text GLabel 1650 4950 0    50   Input ~ 0
 GP4
 $Comp
 L Device:R R4
 U 1 1 61594AFF
-P 8000 4850
-F 0 "R4" V 8207 4850 50  0000 C CNN
-F 1 "330Ω" V 8116 4850 50  0000 C CNN
-F 2 "" V 7930 4850 50  0001 C CNN
-F 3 "~" H 8000 4850 50  0001 C CNN
-	1    8000 4850
+P 1900 4950
+F 0 "R4" V 2107 4950 50  0000 C CNN
+F 1 "330Ω" V 2016 4950 50  0000 C CNN
+F 2 "" V 1830 4950 50  0001 C CNN
+F 3 "~" H 1900 4950 50  0001 C CNN
+	1    1900 4950
 	0    -1   -1   0
 $EndComp
@@
 L Device:LED D2
 U 1 1 61595046
-P 8400 5200
-F 0 "D2" H 8393 4945 50  0000 C CNN
-F 1 "LED" H 8393 5036 50  0000 C CNN
-F 2 "" H 8400 5200 50  0001 C CNN
-F 3 "~" H 8400 5200 50  0001 C CNN
-	1    8400 5200
+P 2300 5300
+F 0 "D2" H 2293 5045 50  0000 C CNN
+F 1 "LED" H 2293 5136 50  0000 C CNN
+F 2 "" H 2300 5300 50  0001 C CNN
+F 3 "~" H 2300 5300 50  0001 C CNN
+	1    2300 5300
 	-1   0    0    1
 $EndComp
-$Comp
-L Device:R R1
-U 1 1 61595C5D
-P 8050 3100
-F 0 "R1" V 7843 3100 50  0000 C CNN
-F 1 "9k8" V 7934 3100 50  0000 C CNN
-F 2 "" V 7980 3100 50  0001 C CNN
-F 3 "~" H 8050 3100 50  0001 C CNN
-	1    8050 3100
-	0    1    1    0
-$EndComp
-Text GLabel 7750 3100 0    50   Input ~ 0
-GND
-Text GLabel 8550 5500 0    50   Input ~ 0
+Text GLabel 2450 5600 0    50   Input ~ 0
 GND
 Wire Wire Line
-	7750 4850 7850 4850
+	1650 4950 1750 4950
 Wire Wire Line
-	8150 4850 8250 4850
+	2050 4950 2150 4950
 Wire Wire Line
-	8550 4850 8650 4850
+	2450 4950 2550 4950
 Wire Wire Line
-	8650 4850 8650 5200
+	2550 4950 2550 5300
 Wire Wire Line
-	8650 5500 8550 5500
+	2550 5600 2450 5600
 Wire Wire Line
-	8550 5200 8650 5200
-Connection ~ 8650 5200
+	2450 5300 2550 5300
+Connection ~ 2550 5300
 Wire Wire Line
-	8650 5200 8650 5500
-Text GLabel 7750 5200 0    50   Input ~ 0
+	2550 5300 2550 5600
+Text GLabel 1650 5300 0    50   Input ~ 0
 SEL
 Text GLabel 8750 2100 2    50   Input ~ 0
@@
 Wire Wire Line
 	8650 2100 8750 2100
-Text GLabel 6450 5400 2    50   Input ~ 0
+Text GLabel 8450 5400 2    50   Input ~ 0
 SW_IN
-Text GLabel 5450 5400 0    50   Input ~ 0
+Text GLabel 7450 5400 0    50   Input ~ 0
 GND
 Wire Wire Line
-	5450 5400 5550 5400
+	7450 5400 7550 5400
 Wire Wire Line
-	6350 5400 6450 5400
+	8350 5400 8450 5400
 Text GLabel 7950 1400 0    50   Input ~ 0
 VBUS
@@
 	8050 1400 8050 1500
 Wire Wire Line
-	7750 5200 8250 5200
+	1650 5300 2150 5300
+Text GLabel 8250 4750 0    50   Input ~ 0
+VBUS
+$Comp
+L Device:R R5
+U 1 1 61508571
+P 8350 5050
+F 0 "R5" H 8420 5096 50  0000 L CNN
+F 1 "10k" H 8420 5005 50  0000 L CNN
+F 2 "" V 8280 5050 50  0001 C CNN
+F 3 "~" H 8350 5050 50  0001 C CNN
+	1    8350 5050
+	1    0    0    -1
+$EndComp
+Connection ~ 8350 5400
 Wire Wire Line
-	8200 3100 8300 3100
+	8250 4750 8350 4750
 Wire Wire Line
-	8300 3100 8300 3350
+	8350 5200 8350 5400
 Wire Wire Line
-	7750 3100 7900 3100
+	8350 4750 8350 4900
+Text GLabel 7800 3950 0    50   Input ~ 0
+SEL
+Text GLabel 7800 3250 0    50   Input ~ 0
+3V3
+Text GLabel 8750 3650 2    50   Input ~ 0
+GP4
+$Comp
+L Device:R R1
+U 1 1 6151ED4F
+P 8100 4300
+F 0 "R1" V 7893 4300 50  0000 C CNN
+F 1 "9k8" V 7984 4300 50  0000 C CNN
+F 2 "" V 8030 4300 50  0001 C CNN
+F 3 "~" H 8100 4300 50  0001 C CNN
+	1    8100 4300
+	0    1    1    0
+$EndComp
+Text GLabel 7800 4300 0    50   Input ~ 0
+GND
 Wire Wire Line
-	7750 3350 8300 3350
-Connection ~ 8300 3350
+	8250 4300 8350 4300
 Wire Wire Line
-	8300 3350 8300 3450
+	7800 4300 7950 4300
 $Comp
 L Transistor_FET:AO3401A Q1
-U 1 1 61652174
-P 8200 3650
-F 0 "Q1" H 8405 3696 50  0000 L CNN
-F 1 "AO3401A" H 8405 3605 50  0000 L CNN
-F 2 "Package_TO_SOT_SMD:SOT-23" H 8400 3575 50  0001 L CIN
-F 3 "http://www.aosmd.com/pdfs/datasheet/AO3401A.pdf" H 8200 3650 50  0001 L CNN
-	1    8200 3650
-	1    0    0    -1
+U 1 1 6151ED6C
+P 8450 3650
+F 0 "Q1" H 8655 3696 50  0000 L CNN
+F 1 "AO3401A" H 8655 3605 50  0000 L CNN
+F 2 "Package_TO_SOT_SMD:SOT-23" H 8650 3575 50  0001 L CIN
+F 3 "http://www.aosmd.com/pdfs/datasheet/AO3401A.pdf" H 8450 3650 50  0001 L CNN
+	1    8450 3650
+	-1   0    0    1
 $EndComp
+$Comp
+L Device:R R2
+U 1 1 615572BC
+P 8100 3250
+F 0 "R2" V 7893 3250 50  0000 C CNN
+F 1 "55Ω" V 7984 3250 50  0000 C CNN
+F 2 "" V 8030 3250 50  0001 C CNN
+F 3 "~" H 8100 3250 50  0001 C CNN
+	1    8100 3250
+	0    1    1    0
+$EndComp
+Wire Wire Line
+	7800 3250 7950 3250
+Wire Wire Line
+	8250 3250 8350 3250
+Wire Wire Line
+	8350 3250 8350 3450
+Wire Wire Line
+	7800 3950 8350 3950
+Wire Wire Line
+	8350 3950 8350 3850
+Wire Wire Line
+	8350 3950 8350 4300
+Connection ~ 8350 3950
+Wire Wire Line
+	8650 3650 8750 3650
 $EndSCHEMATC
