File: KiCAD/MEZ80RAM-SD/MEZ80RAM-SD.kicad_sch (KiCad schematic)
At the start: 21 parts, among them J1 EMUZ80_0, J2 EMUZ80, J3 SD Card slot, J4 ext SPI, U1 Z80CPU, U2 TC551001, U3 MCP23S08-xP

Commit message: Update MEZ80RAM-SD to verion 0.9
Parts:
- removed J3: SD Card slot, Connector_PinSocket_2.54mm:PinSocket_1x06_P2.54mm_Vertical, symbol Connector:Conn_01x06_Socket
- removed R1, R5, R6: 10K, Resistor_SMD:R_0603_1608Metric_Pad0.98x0.95mm_HandSolder, symbol Device:R
- U2: value TC551001 -> AS6C4008; symbol library:TC551001 -> library:AS6C4008
Connections:
- net +5V: now also U1.16 (~{INT}), U3.6 (~{RESET}); no longer U2.30 (CS2)
- net A16: no longer U3.17 (GP7)
- net D2: no longer J4.4 (MISO)
- net ~{CS0}: now also D1.1 (K)
- net A18: now reaches U2.1 (A18)
- net ~{INT} renamed BANK2
- net BANK2: no longer U1.16 (~{INT})
- net ~{LED} renamed BANK1
- net BANK1: no longer D1.1 (K)
- new net A17: U2.30 (A17)
- new net BANK0: U3.17 (GP7)
- new net MISO: J4.4 (MISO)
Other:
- added sheet Untitled Sheet (untitled.kicad_sch)
- title: MEZ80RAM-SD -> SuperMEZ80+SPI
